Commit message: commit 17-03-2017

File: cr_mit/URDF/P102183/urdf/P102183.URDF (robot description, URDF)
Before this commit: robot P102183, 1 links, 0 joints
Links:
- link P102183: geometry collision mesh filename=package://cr_mit/URDF/P102183/meshes/P102183.STL; visual mesh filename=package://cr_mit/URDF/P102183/meshes/P102183.STL

File: cr_mit/URDF/fitting_mjdb9010/urdf/fitting_mjdb9010.URDF (robot description, URDF)
Before this commit: robot fitting_mjdb9010, 1 links, 0 joints
Links:
- link fitting_mjdb9010: geometry collision mesh filename=package://cr_mit/URDF/fitting_mjdb9010/meshes/fitting_mjdb9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; visual mesh filename=package://cr_mit/URDF/fitting_mjdb9010/meshes/fitting_mjdb9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
